File: pcb files (Kicad)/aura-top plate.kicad_pcb (KiCad board)
At the start: 2 copper layers, 36.8 x 47.9 mm, 4 parts

Commit message: moved some things around
Other:
- outline, holes or cut-outs redrawn
